File: hardware/proto_power/proto_power.kicad_pcb (KiCad board)
At the start: 2 copper layers, 60 x 100 mm, 63 parts, among them J1 Trig, J10 Conn_02x08_Odd_Even, J11 Conn_01x03, J12 Conn_01x03, J13 Conn_01x03, J14 Conn_01x03, J2 Conn_01x02_Pin, J3 Gate Out, J4 EG Out, J5 Buffer2 In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

Commit message: v1 board released for mfg.
Parts:
- removed D1: LED, LED_THT:LED_D3.0mm
- removed RV5: 100k, Potentiometer_THT:Potentiometer_Piher_PT-6-V_Vertical
- added R7: 150k, Resistor_THT:R_Axial_DIN0204_L3.6mm_D1.6mm_P2.54mm_Vertical, F.Cu at (106.0, 56.3)
- R8: value 47k -> 120k
- SW2: value GATE -> SW_SPST_LED; footprint Button_Switch_Keyboard:SW_Cherry_MX_1.00u_PCB -> Switches:SW_Cherry_MX_1.00u_Breakout
- moved R5 35.1 mm to (70.5, 76.7), turned to -90 degrees
- moved RV1 35.0 mm to (65.0, 79.0)
- moved R9 31.7 mm to (106.2, 94.2), turned to 90 degrees
- moved SW2 30.0 mm to (97.5, 72.0), turned to 0 degrees
- moved R4 15.6 mm to (80.0, 79.6), turned to 0 degrees
- moved R6 8.02 mm to (106.0, 61.0), turned to 90 degrees
- moved R8 7.17 mm to (108.5, 54.0), turned to 90 degrees
- moved C3 4.05 mm to (82.7, 63.7)
- moved C11 3.05 mm to (76.2, 63.8), turned to 180 degrees
- moved C5 0.51 mm to (68.0, 81.7)
- turned SW1 to 90 degrees
Connections:
- R6 pad 1: Net-(U1-Q) -> Net-(SW2-A)
- R6 pad 2: Net-(D1-A) -> Net-(U1-Q)
Routing:
- net +12V: track 152.3 -> 115.5 mm
- net Net-(D2-K): track 85.9 -> 51.1 mm
- net Net-(J3-PadT): track 7.06 -> 38.9 mm
- net Net-(SW2-A): track 0.00 -> 31.1 mm
- net Net-(Q1-C): track 42.5 -> 66.5 mm
- net Net-(U1-Q): track 53.3 -> 37.3 mm
- net Net-(SW1A-C): track 40.9 -> 56.2 mm, vias 0 -> 2
- net Net-(SW1B-B): track 23.2 -> 16.6 mm
- net Net-(U2A-+): track 45.5 -> 51.7 mm
- net Net-(D1-A): track 3.32 -> 0.00 mm
- net Net-(SW1A-B): track 6.51 -> 5.11 mm
- net +12VRAW: track 147.4 -> 146.3 mm
- net Net-(R5-Pad1): track 8.02 -> 8.96 mm
- net Net-(U1-CV): track 4.39 -> 3.59 mm
- net Net-(Q1-B): track 7.14 -> 6.55 mm
Other:
- board text added: "+12"
- board text added: "+5"
- board text added: "-12"
- board text added: "ATTK"
- board text added: "EG OUT"
- board text added: "GATE"
- board text added: "GATE OUT"
- board text added: "GND"
- board text added: "IN1"
- board text added: "IN2"
- board text added: "MAN"
- board text added: "OSC"
- board text added: "OUT1"
- board text added: "OUT2"
- board text added: "PROTO POWER"
- board text added: "PW/T"
- board text added: "RELS"
- board text added: "TRIG"
- board text added: "Thank yous: Ray Wilson/MFOS, Moritz Klein, Eddy Bergman, Aaron Lanterman"
- board text added: "VOFF"
- board text added: "idyllm CC BY-SA 4.0"
- board text added: "v1.0.20250302"
