File: hardware/proto_power/proto_power.kicad_sch (KiCad schematic)
At the start: 63 parts, among them J1 Trig, J10 Conn_02x08_Odd_Even, J11 Conn_01x03, J12 Conn_01x03, J13 Conn_01x03, J14 Conn_01x03, J2 Conn_01x02_Pin, J3 Gate Out, J4 EG Out, J5 Buffer2 In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

Commit message: v1 board released for mfg.
Parts:
- removed D1: LED, LED_THT:LED_D3.0mm, symbol Device:LED
- removed RV5: 100k, Potentiometer_THT:Potentiometer_Piher_PT-6-V_Vertical, symbol Device:R_Potentiometer_US
- removed SW2: GATE, Button_Switch_Keyboard:SW_Cherry_MX_1.00u_PCB, symbol Switch:SW_Push
- added R7: 150k, Resistor_THT:R_Axial_DIN0204_L3.6mm_D1.6mm_P2.54mm_Vertical, symbol Device:R_US
- added SW2: SW_SPST_LED, Switches:SW_Cherry_MX_1.00u_Breakout, symbol Switch:SW_SPST_LED
- R8: value 47k -> 120k
Connections:
- net GND: now also SW2.1, SW2.3 (K)
- net at Q1.1 (C), R4.2, SW1.6 (C)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: now also SW2.2
- net at R6.1: now also SW2.4 (A); no longer U1.3 (Q)
- net at R6.2: now also U1.3 (Q), R7.1
- net at R8.1, U2.3 (+): now also R7.2
Other:
- company: (none) -> idyllm
- title: (none) -> Prototype Power Module
